File: v0.2.2/mainboardv0.2.2.sch (EAGLE design)
At the start: 17 parts, among them U1 BC127, Y1 MHz

Commit message: Begin the routing
Parts:
- removed U2: (no value), SparkFun-PowerIC:MIC52053.3V
Other:
- moved on the sheet: U1.ANALOG_AUDIO
Changed lines of the file:
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@@
 <part name="GND4" library="supply1" deviceset="GND" device=""/>
 <part name="U1" library="SparkFun-RF" deviceset="BC127" device="" value="BC127"/>
-<part name="U2" library="SparkFun-PowerIC" deviceset="MIC5205" device="3.3V"/>
 <part name="GND5" library="supply1" deviceset="GND" device=""/>
 <part name="S1" library="SparkFun-Electromechanical" deviceset="TAC_SWITCH" device="SMD"/>
@@
 <instance part="C3" gate="G$1" x="-5.08" y="50.8"/>
 <instance part="GND4" gate="1" x="-5.08" y="43.18"/>
-<instance part="U1" gate=".ANALOG_AUDIO" x="142.24" y="-25.4"/>
+<instance part="U1" gate=".ANALOG_AUDIO" x="154.94" y="55.88"/>
 <instance part="U1" gate=".GPIO" x="-50.8" y="63.5"/>
 <instance part="U1" gate=".POWER" x="86.36" y="7.62"/>
 <instance part="U1" gate=".DATA_PORTS" x="86.36" y="68.58"/>
-<instance part="U2" gate="G$1" x="-71.12" y="78.74"/>
 <instance part="GND5" gate="1" x="81.28" y="2.54"/>
 <instance part="S1" gate="S" x="185.42" y="12.7"/>

Commit message: More routing
Parts:
- added C10, C5: 180pF, SparkFun-Capacitors:CAP0603-CAP
- added C11, C13, C6, C8: 0.1uF, SparkFun-Capacitors:0.1UF-25V-5%(0603)
- added C12, C14, C7, C9: 47pF, SparkFun-Capacitors:47PF-50V-5%(0603)
- added C15, C16, C17: 1.0uF, SparkFun-Capacitors:1.0UF-16V-10%(0603)
- added R13, R16, R19, R22: 15K, SparkFun-Resistors:15KOHM1/10W1%(0603)0603
- added R14, R18, R20, R24: 30.1k, SparkFun-Resistors:30.1KOHM1/10W1%(0603)
- added R15, R17, R21, R23: 43k, SparkFun-Resistors:43KOHM1/10W1%(0603)
- added R27: 10K, SparkFun-Resistors:10KOHM1/10W1%(0603)0603
- added U3: TPA6138A2, SparkFun-AnalogIC:TPA6138A2
Connections:
- new net 3.3V: C17.1, R27.1, U3.VDD
- new net L_OUT: C9.1, R18.1, U3.OUTR
- new net N$11: C8.2, R16.2
- new net N$12: C6.2, R13.2
- new net N$13: C5.1, R13.1, R15.2, R18.2
- new net N$14: C9.2, R15.1, U3.INR-
- new net N$15: C7.1, R17.1, U3.INR+
- new net N$16: C5.2, R14.1, R16.1, R17.2
- new net N$17: C10.1, R19.1, R20.2, R21.2
- new net N$18: C12.2, R21.1, U3.INL+
- new net N$19: C11.2, R19.2
- new net N$20: C10.2, R22.1, R23.2, R24.2
- new net N$21: C13.2, R22.2
- new net N$22: C14.2, R23.1, U3.INL-
- new net N$23: R27.2, U3.!MUTE
- new net N$24: C16.1, U3.VSS
- new net N$25: C15.2, U3.CN
- new net N$26: C15.1, U3.CP
- new net R_OUT: C14.1, R24.1, U3.OUTL
- new net SPKR_LN: C6.1, U1.ANALOG_AUDIO.SPKR_LN
- new net SPKR_LP: C8.1, U1.ANALOG_AUDIO.SPKR_LP
- new net SPKR_RN: C13.1, U1.ANALOG_AUDIO.SPKR_RN
- new net SPKR_RP: C11.1, U1.ANALOG_AUDIO.SPKR_RP
- net GND: now also C12.1, C16.2, C17.2, C7.2, R14.2, R20.1, U3.GND
Other:
- moved on the sheet: U1.ANALOG_AUDIO
