File: vf0.1/mainboard_reciever.vf0.1.brd (EAGLE design)
At the start: 48.9 x 38.4 mm, 17 parts, among them J1 AVR_SPI_PRG_6TESTPOINTS, J2 U.FL, Y1 16MHz

Commit message: Add everything
Parts:
- removed L, R: RCA, SparkFun-Connectors:RCA
- removed SI4713_BREAKOUT: M11PTH, SparkFun-Connectors:1X11
- added C5: 1uF, SparkFun-Capacitors:0603-CAP
- added C6: (no value), SparkFun-Capacitors:CPOL-RADIAL-10UF-25V
- added C7: (no value), SparkFun-Capacitors:0603-CAP
- added D1: GREEN, SparkFun-LED:LED-0603
- added J3: U.FL, SparkFun-Connectors:U.FL
- added JP2: (no value), SparkFun-Connectors:AUDIO-JACK
- added JP3: (no value), SparkFun-Connectors:1X08_PIN1_NO_SILK
- added R4: 1K, SparkFun-Resistors:0603-RES
- added S1: (no value), SparkFun-Electromechanical:SWITCH-SPDT-SMD
- added U1: MAX1555, SparkFun-PowerIC:SOT23-5
- C1, C4: device SparkFun-Capacitors:CAP-PTH-SMALL -> SparkFun-Capacitors:0603-CAP
- J2: value U.FL -> (none); device SparkFun-Connectors:U.FL -> SparkFun-Connectors:JST-2-SMD
- R1, R2, R3: device SparkFun-Resistors:AXIAL-0.1 -> SparkFun-Resistors:0603-RES
- U$2: value RF-LINK_TX -> 3.3V/150mA; device SparkFun-RF:RF-LINK_TX -> SparkFun-PowerIC:SOT23-5
- U$3: value (none) -> RF-LINK_RX; device SparkFun-Aesthetics:OSHW-LOGO-L -> SparkFun-RF:RF-LINK_RX
- moved U$3 43.5 mm to (47.9, 6.35), turned to 180 degrees
- moved J2 31.4 mm to (27.9, 29.8), turned to 270 degrees
- moved U$2 30.6 mm to (11.7, 29.2), turned to 90 degrees
- moved C1 11.1 mm to (19.4, 22.1)
- moved R3 4.33 mm to (27.2, 10.5), turned to 0 degrees
- moved C4 3.06 mm to (19.4, 16.0), turned to 180 degrees
- moved R1 1.67 mm to (19.4, 20.1)
- moved R2 1.65 mm to (19.4, 18.0)
Connections:
- removed net RADIODAT: U$1.25, U$2.DATA
- removed net SCL: SI4713_BREAKOUT.9, U$1.18
- removed net SDA: SI4713_BREAKOUT.8, U$1.19
- removed net T_RST: SI4713_BREAKOUT.11, U$1.26
- new net N$10: R4.1, U1.3
- new net N$11: S1.1, U$2.1, U$2.3
- new net N$12: J3.P$3, U$3.ANT
- new net N$8: C5.1, D1.A, J2.2, S1.2, U1.5
- new net UVCC: C4.1, JP1.VBUS, U$1.2, U$1.7, U1.1
- net !RESET: now also R3.1; no longer R3.P$1
- net GND: now also C5.2, C6.2, C7.2, J2.1, J3.P$1, J3.P$2, JP2.SLEEVE, JP3.7, U$2.2, U$3.GND@1, U1.2; no longer J2.P$1, J2.P$2, L.PIN, R.PIN, SI4713_BREAKOUT.4, U$2.GND
- net L: now also JP2.TIP; no longer L.SHELL, SI4713_BREAKOUT.2
- net N$1: now also R2.1; no longer R2.P$1
- net N$2: now also R1.1; no longer R1.P$1
- net N$3: now also R1.2; no longer R1.P$2
- net N$4: now also R2.2; no longer R2.P$2
- net N$9: now also D1.C, R4.2; no longer J2.P$3, U$2.ANT
- net R: now also JP2.RING; no longer R.SHELL, SI4713_BREAKOUT.1
- net VCC: now also C6.1, C7.1, R3.2, U$2.5, U$3.+5V@1; no longer C4.1, JP1.VBUS, R3.P$2, SI4713_BREAKOUT.3, U$1.2, U$1.7, U$2.VCC
Routing:
- net L: track 51.8 -> 0.00 mm
- net VCC: track 82.0 -> 30.3 mm, vias 0 -> 2
- net R: track 42.2 -> 0.00 mm
- net UVCC: track 0.00 -> 36.3 mm, vias 0 -> 1
- net SCL: track 30.2 -> 0.00 mm, vias 1 -> 0
- net N$8: track 0.00 -> 28.4 mm
- net SDA: track 27.2 -> 0.00 mm, vias 1 -> 0
- net T_RST: track 19.2 -> 0.00 mm
- net RADIODAT: track 12.7 -> 0.00 mm, vias 1 -> 0
- net N$11: track 0.00 -> 9.91 mm
- net N$9: track 7.49 -> 1.63 mm
- net N$12: track 0.00 -> 5.58 mm
- net N$10: track 0.00 -> 4.59 mm
- net !RESET: track 12.5 -> 9.27 mm
- net N$5: track 9.61 -> 6.81 mm, vias 1 -> 2
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Other:
- board text removed: "DAT"

Commit message: Reciever stuff. Not done yet :)
Parts:
- added D2: BLUE, SparkFun-LED:LED-0603
- added JP4: AUDIOIN, SparkFun-Connectors:1X03
- added R5: 1K, SparkFun-Resistors:0603-RES
- added S2, S3: SWITCH-MOMENTARY-2SIDE_EZ, SparkFun-Electromechanical:TACTILE-PTH-SIDEEZ
- added U$4: (no value), SparkFun-Aesthetics:OSHW-LOGO-L
- C2, C3: device SparkFun-Capacitors:CAP-PTH-SMALL -> SparkFun-Capacitors:0603-CAP
- C6: value (none) -> 10uF
- C7: value (none) -> 0.1uF
- J2: value (none) -> BATTERY
- JP1: value USB-B -> USBSMD; device SparkFun-Connectors:USB-B-PTH -> SparkFun-Connectors:USB-MINIB
- JP2: value (none) -> HEADPHONES
- S1: value (none) -> POWERSWITCH
- Y1: device SparkFun-FreqCtrl:HC49US -> SparkFun-FreqCtrl:CRYSTAL-SMD-5X3
- moved U$3 42.7 mm to (5.33, 10.0), turned to 0 degrees
- moved J3 28.3 mm to (35.8, 16.3), turned to 270 degrees
- moved R3 6.36 mm to (20.8, 10.3)
- moved J1 5.99 mm to (24.1, 17.8)
- moved U$1 5.86 mm to (24.1, 17.8)
- moved R1 5.10 mm to (14.6, 18.4)
- moved R2 4.91 mm to (14.6, 17.1)
- moved C4 4.83 mm to (14.6, 15.7)
- moved C3 4.77 mm to (22.1, 7.11), turned to 90 degrees
- moved C2 4.67 mm to (26.9, 7.11), turned to 270 degrees
- moved JP2 4.44 mm to (45.7, 21.6)
- moved JP1 3.98 mm to (8.51, 17.9)
- moved C1 2.95 mm to (16.8, 23.4)
- moved J2 2.67 mm to (25.3, 29.7)
- moved Y1 1.20 mm to (24.5, 7.62), turned to 270 degrees
- renumbered JP3 to SI4703_TUNER
Connections:
- new net !RST: SI4703_TUNER.3, U$1.26
- new net BLINKY: D2.A, U$1.32
- new net N$14: D2.C, R5.1
- new net RDAT: U$1.31, U$3.DATA@1
- new net SCL: SI4703_TUNER.5, U$1.18
- new net SDA: SI4703_TUNER.6, U$1.19
- new net V_DWN: S3.1, U$1.29
- new net V_UP: S2.1, U$1.28
- net GND: now also JP4.1, R5.2, S2.2, S3.2
- net L: now also JP4.2
- net N$6: now also Y1.3; no longer Y1.2
- net R: now also JP4.3
- net VCC: now also SI4703_TUNER.8
Routing:
- net VCC: track 30.3 -> 75.8 mm
- net RDAT: track 0.00 -> 36.0 mm, vias 0 -> 1
- net V_DWN: track 0.00 -> 35.6 mm, vias 0 -> 1
- net SCL: track 0.00 -> 29.3 mm, vias 0 -> 1
- net GND: track 25.7 -> 54.2 mm, vias 7 -> 9
- net SDA: track 0.00 -> 25.8 mm, vias 0 -> 1
- net !RST: track 0.00 -> 22.4 mm
- net V_UP: track 0.00 -> 20.3 mm, vias 0 -> 1
- net R: track 0.00 -> 19.1 mm
- net N$7: track 15.2 -> 4.55 mm
- net N$12: track 5.58 -> 13.6 mm
- net L: track 0.00 -> 6.99 mm
- net BLINKY: track 0.00 -> 5.46 mm
- net N$1: track 7.52 -> 3.06 mm
- net UVCC: track 36.3 -> 32.3 mm, vias 1 -> 3
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Other:
- board size 48.9 x 38.4 mm -> 43.8 x 34.6 mm
