File: vf0.1/mainboard_reciever.vf0.1.sch (EAGLE design)
At the start: 16 parts, among them J1 AVR_SPI_PRG_6TESTPOINTS, J2 U.FL, Y1 16MHz

Commit message: Add everything
Parts:
- removed L, R: RCA, SparkFun-Connectors:RCA
- removed SI4713_BREAKOUT: M11PTH, SparkFun-Connectors:M11PTH
- added C5: 1uF, SparkFun-Capacitors:1.0UF-16V-10%(0603)
- added C6: (no value), SparkFun-Capacitors:10UF-25V-20%(PTH)
- added C7: (no value), SparkFun-Capacitors:0.1UF-25V(+80/-20%)(0603)
- added D1: GREEN, SparkFun-LED:LED-GREEN0603
- added J3: U.FL, SparkFun-Connectors:U.FL
- added JP2: (no value), SparkFun-Connectors:AUDIO-JACKPTH
- added JP3: (no value), SparkFun-Connectors:M08
- added R4: 1K, SparkFun-Resistors:1KOHM1/10W1%(0603)
- added S1: (no value), SparkFun-Electromechanical:SWITCH-SPDTSMD2
- added U$3: RF-LINK_RX, SparkFun-RF:RF-LINK_RX
- added U1: MAX1555, SparkFun-PowerIC:MAX1555
- C1, C4: device SparkFun-Capacitors:CAPPTH -> SparkFun-Capacitors:CAP0603-CAP
- J2: value U.FL -> (none); device SparkFun-Connectors:U.FL -> SparkFun-Connectors:JST_2MM_MALE
- R1, R2: device SparkFun-Resistors:RESISTORPTH-1/4W-VERT -> SparkFun-Resistors:RESISTOR0603
- R3: device SparkFun-Resistors:10KOHM-1/4W5%(PTH)VERT -> SparkFun-Resistors:10KOHM1/10W1%(0603)0603
- U$2: value RF-LINK_TX -> 3.3V/150mA; device SparkFun-RF:RF-LINK_TX -> SparkFun-PowerIC:V_REG_MIC52053.3V
Connections:
- removed net RADIODAT: U$1.PD4(ADC8), U$2.DATA
- removed net SCL: SI4713_BREAKOUT.9, U$1.PD0(SCL)
- removed net SDA: SI4713_BREAKOUT.8, U$1.PD1(SDA)
- removed net T_RST: SI4713_BREAKOUT.11, U$1.PD6(ADC9)
- new net N$10: R4.1, U1.CHG
- new net N$11: S1.O, U$2.EN, U$2.IN
- new net N$12: J3.SIGNAL, U$3.ANT
- new net N$8: C5.1, D1.A, J2.+, S1.P, U1.BATT
- new net UVCC: C4.1, JP1.VBUS, U$1.UVCC, U$1.VBUS, U1.USB
- net GND: now also C5.2, C6.-, C7.2, J2.-, J3.GND@0, J3.GND@1, JP2.SLEEVE, JP3.7, U$3.GND, U1.GND; no longer J2.GND@0, J2.GND@1, L.PIN, R.PIN, SI4713_BREAKOUT.4
- net L: now also JP2.LEFT; no longer L.SHELL, SI4713_BREAKOUT.2
- net N$9: now also D1.C, R4.2; no longer J2.SIGNAL, U$2.ANT
- net R: now also JP2.RIGHT; no longer R.SHELL, SI4713_BREAKOUT.1
- net VCC: now also C6.+, C7.1, U$2.OUT, U$3.+5V; no longer C4.1, JP1.VBUS, SI4713_BREAKOUT.3, U$1.UVCC, U$1.VBUS, U$2.+5V
Other:
- note added: "ATmega32u4 microcontroller"
- note added: "Audio Connection"
- note added: "ISP connection"
- note added: "USB connection"

Commit message: Reciever stuff. Not done yet :)
Parts:
- added D2: BLUE, SparkFun-LED:LED-BLUE0603
- added JP4: AUDIOIN, SparkFun-Connectors:M03PTH
- added R5: 1K, SparkFun-Resistors:1KOHM1/10W1%(0603)
- added S2, S3: SWITCH-MOMENTARY-2SIDE_EZ, SparkFun-Electromechanical:SWITCH-MOMENTARY-2SIDE_EZ
- C2, C3: device SparkFun-Capacitors:CAPPTH -> SparkFun-Capacitors:CAP0603-CAP
- C6: value (none) -> 10uF
- C7: value (none) -> 0.1uF
- J2: value (none) -> BATTERY
- JP1: value USB-B -> USBSMD; device SparkFun-Connectors:USBPTH -> SparkFun-Connectors:USBSMD
- JP2: value (none) -> HEADPHONES
- S1: value (none) -> POWERSWITCH
- Y1: device SparkFun-FreqCtrl:CRYSTALHC49US -> SparkFun-FreqCtrl:CRYSTAL5X3
- renumbered JP3 to SI4703_TUNER
Connections:
- new net !RST: SI4703_TUNER.3, U$1.PD6(ADC9)
- new net BLINKY: D2.A, U$1.PC7
- new net N$14: D2.C, R5.1
- new net RDAT: U$1.PC6, U$3.DATA
- new net SCL: SI4703_TUNER.5, U$1.PD0(SCL)
- new net SDA: SI4703_TUNER.6, U$1.PD1(SDA)
- new net V_DWN: S3.1, U$1.PB5(ADC12)
- new net V_UP: S2.1, U$1.PB4(ADC11)
- net GND: now also JP4.1, R5.2, S2.2, S3.2
- net L: now also JP4.2
- net R: now also JP4.3
- net VCC: now also SI4703_TUNER.8
Other:
- note added: "Battery Charger and Power Supply"
- note added: "Das Blinkenlichten"
- note added: "Data Radio"
- note added: "FM Tuner"
- note added: "Volume buttons"
- moved on the sheet: J3, U$3
